File: BasePlate.brd (EAGLE design)
At the start: 292.2 x 120 mm, 7 parts

Commit message: remove support for old gimbals
Parts:
- removed E$1, E$2: (no value), RemotePartsA:GIMBAL_FOOTPRINT_SCREWS
Other:
- outline, holes or cut-outs redrawn
Changed lines of the file:
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@@
 <wire x1="-93" y1="60" x2="-33" y2="60" width="0.0254" layer="20"/>
 <wire x1="-33" y1="60" x2="-28" y2="55" width="0.0254" layer="20" curve="-90"/>
-<wire x1="-28" y1="55" x2="-28" y2="-6" width="0.0254" layer="20"/>
-<wire x1="-28" y1="-6" x2="-23" y2="-11" width="0.0254" layer="20" curve="90"/>
-<wire x1="-23" y1="-11" x2="25" y2="-11" width="0.0254" layer="20"/>
-<wire x1="25" y1="-11" x2="30" y2="-6" width="0.0254" layer="20" curve="90"/>
-<wire x1="30" y1="-6" x2="30" y2="55" width="0.0254" layer="20"/>
+<wire x1="-19" y1="0" x2="-23" y2="0" width="0.0254" layer="20"/>
+<wire x1="-23" y1="0" x2="-28" y2="5" width="0.0254" layer="20" curve="-90"/>
+<wire x1="-28" y1="5" x2="-28" y2="55" width="0.0254" layer="20"/>
+<wire x1="-9" y1="-11" x2="9" y2="-11" width="0.0254" layer="20"/>
+<wire x1="9" y1="-11" x2="14" y2="-6" width="0.0254" layer="20" curve="90"/>
+<wire x1="14" y1="-6" x2="14" y2="-5" width="0.0254" layer="20"/>
+<wire x1="14" y1="-5" x2="19" y2="0" width="0.0254" layer="20" curve="-90"/>
+<wire x1="19" y1="0" x2="25" y2="0" width="0.0254" layer="20"/>
+<wire x1="25" y1="0" x2="30" y2="5" width="0.0254" layer="20" curve="90"/>
+<wire x1="30" y1="5" x2="30" y2="55" width="0.0254" layer="20"/>
+<wire x1="-9" y1="-11" x2="-14" y2="-6" width="0.0254" layer="20" curve="-90"/>
+<wire x1="-14" y1="-6" x2="-14" y2="-5" width="0.0254" layer="20"/>
 <wire x1="30" y1="55" x2="35" y2="60" width="0.0254" layer="20" curve="-90"/>
 <wire x1="35" y1="60" x2="93" y2="60" width="0.0254" layer="20"/>
@@
 <wire x1="146" y1="0" x2="93" y2="60" width="0.0254" layer="20" curve="90"/>
 <dimension x1="-146" y1="0" x2="146" y2="0" x3="0" y3="61" textsize="1.778" layer="47" dtype="horizontal" unit="inch"/>
-<wire x1="-90" y1="19" x2="-78" y2="19" width="0.0254" layer="20"/>
-<wire x1="-78" y1="19" x2="-76" y2="17" width="0.0254" layer="20" curve="-90"/>
-<wire x1="-76" y1="17" x2="-76" y2="-17" width="0.0254" layer="20"/>
-<wire x1="-76" y1="-17" x2="-78" y2="-19" width="0.0254" layer="20" curve="-90"/>
-<wire x1="-78" y1="-19" x2="-90" y2="-19" width="0.0254" layer="20"/>
-<wire x1="-90" y1="-19" x2="-92" y2="-21" width="0.0254" layer="20" curve="90"/>
-<wire x1="-92" y1="-21" x2="-92" y2="-23" width="0.0254" layer="20"/>
-<wire x1="-92" y1="25" x2="-92" y2="21" width="0.0254" layer="20"/>
-<wire x1="-92" y1="21" x2="-90" y2="19" width="0.0254" layer="20" curve="90"/>
-<wire x1="-92" y1="25" x2="-94" y2="27" width="0.0254" layer="20" curve="90"/>
-<wire x1="-94" y1="27" x2="-130" y2="27" width="0.0254" layer="20"/>
-<wire x1="-130" y1="27" x2="-132" y2="25" width="0.0254" layer="20" curve="90"/>
-<wire x1="-132" y1="25" x2="-132" y2="21" width="0.0254" layer="20"/>
-<wire x1="-132" y1="21" x2="-134" y2="19" width="0.0254" layer="20" curve="-90"/>
-<wire x1="-134" y1="19" x2="-135" y2="19" width="0.0254" layer="20"/>
-<wire x1="-135" y1="-19" x2="-134" y2="-19" width="0.0254" layer="20"/>
-<wire x1="-134" y1="-19" x2="-132" y2="-21" width="0.0254" layer="20" curve="-90"/>
-<wire x1="-132" y1="-21" x2="-132" y2="-23" width="0.0254" layer="20"/>
-<wire x1="-132" y1="-23" x2="-130" y2="-25" width="0.0254" layer="20" curve="90"/>
-<wire x1="-130" y1="-25" x2="-94" y2="-25" width="0.0254" layer="20"/>
-<wire x1="-94" y1="-25" x2="-92" y2="-23" width="0.0254" layer="20" curve="90"/>
-<wire x1="-135" y1="19" x2="-137" y2="17" width="0.0254" layer="20" curve="90"/>
-<wire x1="-137" y1="17" x2="-137" y2="-17" width="0.0254" layer="20"/>
-<wire x1="-137" y1="-17" x2="-135" y2="-19" width="0.0254" layer="20" curve="90"/>
-<wire x1="90" y1="-19" x2="77" y2="-19" width="0.0254" layer="20"/>
-<wire x1="77" y1="-19" x2="75" y2="-17" width="0.0254" layer="20" curve="-90"/>
-<wire x1="75" y1="-17" x2="75" y2="17" width="0.0254" layer="20"/>
-<wire x1="75" y1="17" x2="77" y2="19" width="0.0254" layer="20" curve="-90"/>
-<wire x1="77" y1="19" x2="90" y2="19" width="0.0254" layer="20"/>
-<wire x1="90" y1="19" x2="92" y2="21" width="0.0254" layer="20" curve="90"/>
-<wire x1="92" y1="21" x2="92" y2="23" width="0.0254" layer="20"/>
-<wire x1="92" y1="-25" x2="92" y2="-21" width="0.0254" layer="20"/>
-<wire x1="92" y1="-21" x2="90" y2="-19" width="0.0254" layer="20" curve="90"/>
-<wire x1="92" y1="-25" x2="94" y2="-27" width="0.0254" layer="20" curve="90"/>
-<wire x1="94" y1="-27" x2="130" y2="-27" width="0.0254" layer="20"/>
-<wire x1="130" y1="-27" x2="132" y2="-25" width="0.0254" layer="20" curve="90"/>
-<wire x1="132" y1="-25" x2="132" y2="-21" width="0.0254" layer="20"/>
-<wire x1="132" y1="-21" x2="134" y2="-19" width="0.0254" layer="20" curve="-90"/>
-<wire x1="134" y1="-19" x2="135" y2="-19" width="0.0254" layer="20"/>
-<wire x1="135" y1="19" x2="134" y2="19" width="0.0254" layer="20"/>
-<wire x1="134" y1="19" x2="132" y2="21" width="0.0254" layer="20" curve="-90"/>
-<wire x1="132" y1="21" x2="132" y2="23" width="0.0254" layer="20"/>
-<wire x1="132" y1="23" x2="130" y2="25" width="0.0254" layer="20" curve="90"/>
-<wire x1="130" y1="25" x2="94" y2="25" width="0.0254" layer="20"/>
-<wire x1="94" y1="25" x2="92" y2="23" width="0.0254" layer="20" curve="90"/>
-<wire x1="135" y1="-19" x2="137" y2="-17" width="0.0254" layer="20" curve="90"/>
-<wire x1="137" y1="-17" x2="137" y2="17" width="0.0254" layer="20"/>
-<wire x1="137" y1="17" x2="135" y2="19" width="0.0254" layer="20" curve="90"/>
+<wire x1="-76" y1="-21" x2="-76" y2="21" width="0.0254" layer="20"/>
+<wire x1="-76" y1="21" x2="-78" y2="23" width="0.0254" layer="20" curve="90"/>
+<wire x1="-78" y1="23" x2="-83" y2="23" width="0.0254" layer="20"/>
+<wire x1="-83" y1="23" x2="-85" y2="25" width="0.0254" layer="20" curve="-90"/>
+<wire x1="-85" y1="25" x2="-85" y2="26" width="0.0254" layer="20"/>
+<wire x1="-85" y1="26" x2="-87" y2="28" width="0.0254" layer="20" curve="90"/>
+<wire x1="-87" y1="28" x2="-129" y2="28" width="0.0254" layer="20"/>
+<wire x1="-83" y1="-23" x2="-78" y2="-23" width="0.0254" layer="20"/>
+<wire x1="-78" y1="-23" x2="-76" y2="-21" width="0.0254" layer="20" curve="90"/>
+<wire x1="-85" y1="-26" x2="-85" y2="-25" width="0.0254" layer="20"/>
+<wire x1="-85" y1="-25" x2="-83" y2="-23" width="0.0254" layer="20" curve="-90"/>
+<wire x1="-135" y1="-23" x2="-133" y2="-23" width="0.0254" layer="20"/>
+<wire x1="-133" y1="-23" x2="-131" y2="-25" width="0.0254" layer="20" curve="-90"/>
+<wire x1="-131" y1="-25" x2="-131" y2="-26" width="0.0254" layer="20"/>
+<wire x1="-131" y1="-26" x2="-129" y2="-28" width="0.0254" layer="20" curve="90"/>
+<wire x1="-129" y1="-28" x2="-87" y2="-28" width="0.0254" layer="20"/>
+<wire x1="-87" y1="-28" x2="-85" y2="-26" width="0.0254" layer="20" curve="90"/>
+<wire x1="-129" y1="28" x2="-131" y2="26" width="0.0254" layer="20" curve="90"/>
+<wire x1="-131" y1="26" x2="-131" y2="25" width="0.0254" layer="20"/>
+<wire x1="-131" y1="25" x2="-133" y2="23" width="0.0254" layer="20" curve="-90"/>
+<wire x1="-133" y1="23" x2="-135" y2="23" width="0.0254" layer="20"/>
+<wire x1="-135" y1="23" x2="-137" y2="21" width="0.0254" layer="20" curve="90"/>
+<wire x1="-137" y1="21" x2="-137" y2="-21" width="0.0254" layer="20"/>
+<wire x1="-137" y1="-21" x2="-135" y2="-23" width="0.0254" layer="20" curve="90"/>
+<wire x1="77" y1="-23" x2="83" y2="-23" width="0.0254" layer="20"/>
+<wire x1="83" y1="-23" x2="85" y2="-25" width="0.0254" layer="20" curve="-90"/>
+<wire x1="85" y1="-25" x2="85" y2="-26" width="0.0254" layer="20"/>
+<wire x1="85" y1="-26" x2="87" y2="-28" width="0.0254" layer="20" curve="90"/>
+<wire x1="87" y1="-28" x2="130" y2="-28" width="0.0254" layer="20"/>
+<wire x1="130" y1="-28" x2="132" y2="-26" width="0.0254" layer="20" curve="90"/>
+<wire x1="132" y1="-26" x2="132" y2="-25" width="0.0254" layer="20"/>
+<wire x1="132" y1="-25" x2="134" y2="-23" width="0.0254" layer="20" curve="-90"/>
+<wire x1="134" y1="-23" x2="135" y2="-23" width="0.0254" layer="20"/>
+<wire x1="135" y1="-23" x2="137" y2="-21" width="0.0254" layer="20" curve="90"/>
+<wire x1="137" y1="-21" x2="137" y2="21" width="0.0254" layer="20"/>
+<wire x1="137" y1="21" x2="135" y2="23" width="0.0254" layer="20" curve="90"/>
+<wire x1="135" y1="23" x2="133" y2="23" width="0.0254" layer="20"/>
+<wire x1="133" y1="23" x2="131" y2="25" width="0.0254" layer="20" curve="-90"/>
+<wire x1="131" y1="25" x2="131" y2="26" width="0.0254" layer="20"/>
+<wire x1="75" y1="21" x2="75" y2="-21" width="0.0254" layer="20"/>
+<wire x1="75" y1="-21" x2="77" y2="-23" width="0.0254" layer="20" curve="90"/>
+<wire x1="83" y1="23" x2="77" y2="23" width="0.0254" layer="20"/>
+<wire x1="77" y1="23" x2="75" y2="21" width="0.0254" layer="20" curve="90"/>
+<wire x1="131" y1="26" x2="129" y2="28" width="0.0254" layer="20" curve="90"/>
+<wire x1="129" y1="28" x2="87" y2="28" width="0.0254" layer="20"/>
+<wire x1="87" y1="28" x2="85" y2="26" width="0.0254" layer="20" curve="90"/>
+<wire x1="85" y1="26" x2="85" y2="25" width="0.0254" layer="20"/>
+<wire x1="85" y1="25" x2="83" y2="23" width="0.0254" layer="20" curve="-90"/>
+<wire x1="-14" y1="-5" x2="-19" y2="0" width="0.0254" layer="20" curve="90"/>
 </plain>
 <attributes>
@@
 </autorouter>
 <elements>
-<element name="E$1" library="RemotePartsA" package="GIMBAL_FOOTPRINT_SCREWS" value="" x="-112" y="0" locked="yes"/>
-<element name="E$2" library="RemotePartsA" package="GIMBAL_FOOTPRINT_SCREWS" value="" x="112" y="0" locked="yes" rot="R180"/>
 <element name="E$3" library="RemotePartsA" package="FRSKY-TARANIS-GIMBAL" value="" x="-108" y="0" locked="yes"/>
 <element name="E$4" library="RemotePartsA" package="FRSKY-TARANIS-GIMBAL" value="" x="108" y="0" locked="yes" rot="R180"/>
