File: hardware/controller_board.sch (EAGLE design)
At the start: 47 parts, among them J1 FRSKY-GIMBAL, J2 FRSKY-GIMBAL, J3 WIRE-HARNESS-SPARKFUN-9915, J4 AVR_SPI_PRG_6NS, J7 FTDI_BASICPTH, U1 ATMEGA128RFA1, U2 TPS73633-DBVT, Y1 CRYSTAL5X3

Commit message: Remove big caps
Parts:
- removed C2, C7: (no value), KoalaBuild:RESOLVED-CAPACITOR-POL_TH-RADIAL_ALUMINUM_6.3MM
Connections:
- net +3V3: no longer C2.+
- net GND: no longer C2.-, C7.-
- net VBAT: no longer C7.+
Changed lines of the file:
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@@
 <?xml version="1.0" encoding="utf-8"?>
 <!DOCTYPE eagle SYSTEM "eagle.dtd">
-<eagle version="7.6.0">
+<eagle version="9.0.0">
 <drawing>
 <settings>
 <setting alwaysvectorfont="no"/>
+<setting keepoldvectorfont="yes"/>
 <setting verticaltext="up"/>
 </settings>
@@
 </part>
 <part name="+3V7" library="supply1" deviceset="+3V3" device=""/>
-<part name="C2" library="KoalaBuild" deviceset="RESOLVED-CAPACITOR-POL_" device="TH-RADIAL_ALUMINUM_6.3MM">
-<attribute name="DIST" value="Digikey"/>
-<attribute name="DISTPN" value="P5152-ND"/>
-</part>
 <part name="GND10" library="supply1" deviceset="GND" device=""/>
 <part name="TM3" library="RemoteParts" deviceset="TRIMPOT" device="3386"/>
@@
 <part name="GND25" library="supply1" deviceset="GND" device=""/>
 <part name="P+4" library="quadparts_prebuilt" deviceset="VBAT" device=""/>
-<part name="C7" library="KoalaBuild" deviceset="RESOLVED-CAPACITOR-POL_" device="TH-RADIAL_ALUMINUM_6.3MM">
-<attribute name="DIST" value="Digikey"/>
-<attribute name="DISTPN" value="P5152-ND"/>
-</part>
-<part name="GND1" library="quadparts_prebuilt" deviceset="GND" device=""/>
-<part name="GND3" library="quadparts_prebuilt" deviceset="GND" device=""/>
 <part name="R4" library="quadparts_prebuilt" deviceset="RESISTOR_" device="SMD-2012-0805-10K" value="10K"/>
 <part name="R5" library="quadparts_prebuilt" deviceset="RESISTOR_" device="SMD-2012-0805-10K" value="10K"/>
@@
 <instance part="3.3V" gate="G$1" x="294.64" y="30.48"/>
 <instance part="+3V7" gate="G$1" x="304.8" y="45.72"/>
-<instance part="C2" gate="G$1" x="309.88" y="-12.7"/>
 <instance part="GND10" gate="1" x="66.04" y="147.32"/>
 <instance part="TM3" gate="G$1" x="134.62" y="157.48"/>
@@
 <instance part="GND25" gate="1" x="259.08" y="0"/>
 <instance part="P+4" gate="VCC" x="266.7" y="12.7"/>
-<instance part="C7" gate="G$1" x="251.46" y="7.62"/>
-<instance part="GND1" gate="1" x="309.88" y="-20.32"/>
-<instance part="GND3" gate="1" x="251.46" y="0"/>
 <instance part="R4" gate="G$1" x="10.16" y="106.68" rot="R90"/>
 <instance part="R5" gate="G$1" x="10.16" y="96.52" rot="R90"/>
@@
 </segment>
 <segment>
-<pinref part="C2" gate="G$1" pin="-"/>
-<pinref part="GND1" gate="1" pin="GND"/>
-</segment>
-<segment>
-<pinref part="C7" gate="G$1" pin="-"/>
-<pinref part="GND3" gate="1" pin="GND"/>
-</segment>
-<segment>
 <pinref part="R5" gate="G$1" pin="1"/>
 <pinref part="GND12" gate="1" pin="GND"/>
@@
 <wire x1="297.18" y1="-7.62" x2="297.18" y2="-10.16" width="0.1524" layer="91"/>
 <junction x="302.26" y="-10.16"/>
-<pinref part="C2" gate="G$1" pin="+"/>
-<wire x1="309.88" y1="-10.16" x2="302.26" y2="-10.16" width="0.1524" layer="91"/>
 <pinref part="D4" gate="G$1" pin="A"/>
-<wire x1="309.88" y1="-10.16" x2="317.5" y2="-10.16" width="0.1524" layer="91"/>
-<junction x="309.88" y="-10.16"/>
+<wire x1="302.26" y1="-10.16" x2="317.5" y2="-10.16" width="0.1524" layer="91"/>
 </segment>
 <segment>
@@
 <segment>
 <pinref part="C16" gate="G$1" pin="1"/>
-<junction x="259.08" y="10.16"/>
 <pinref part="U2" gate="G$1" pin="EN"/>
 <wire x1="266.7" y1="10.16" x2="259.08" y2="10.16" width="0.1524" layer="91"/>
@@
 <pinref part="S1" gate="G$1" pin="C"/>
 <pinref part="P+4" gate="VCC" pin="VBAT"/>
-<pinref part="C7" gate="G$1" pin="+"/>
-<wire x1="259.08" y1="10.16" x2="251.46" y2="10.16" width="0.1524" layer="91"/>
-</segment>
-<segment>
+</segment>
+<segment>
