File: hardware/power_test.brd (EAGLE design)
At the start: 45.2 x 49.3 mm, 46 parts, among them J10 USB-MICROA-AMPHENOL-10118192-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, J3 USB-MICROB-EDAC-690-005-299-0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, U1 DPDT-X2, U3 FT232RLSSOP, U4 MCP73831T-2ACI/OT

Commit message: Set charging current to 450mA
Parts:
- removed R2: 10K, quadparts_prebuilt:RESC2012X60_HS
- R10: value 2K -> 2.2K
Connections:
- removed net CHR_ENABLE#: R10.2, R2.2, U3.14
- net 3V3: no longer R2.1
- net GND: now also R10.2
Changed lines of the file:
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@@
 <attribute name="DIST" value="Digikey" x="-41.7331" y="14.312940625" size="1.778" layer="27" display="off"/>
 <attribute name="DISTPN" value="3M9448-ND" x="-41.7331" y="14.312940625" size="1.778" layer="27" display="off"/>
+<attribute name="NAME" x="-39.1931" y="9.272940625" size="1.778" layer="51" font="vector" ratio="10" align="center"/>
 <attribute name="NAME" x="-39.1931" y="12.172940625" size="1.27" layer="25" font="vector" ratio="10" align="center"/>
-<attribute name="NAME" x="-39.1931" y="9.272940625" size="1.778" layer="51" font="vector" ratio="10" align="center"/>
 <attribute name="PIN1" value="" x="-41.7331" y="16.217940625" size="1.778" layer="21" font="vector" rot="R90" align="center-left"/>
 <attribute name="PIN2" value="" x="-39.1931" y="16.217940625" size="1.778" layer="21" font="vector" rot="R90" align="center-left"/>
@@
 <attribute name="DIST" value="Digikey" x="-33.39758125" y="14.34221875" size="1.778" layer="27" display="off"/>
 <attribute name="DISTPN" value="3M9448-ND" x="-33.39758125" y="14.34221875" size="1.778" layer="27" display="off"/>
+<attribute name="NAME" x="-30.35758125" y="9.30221875" size="1.778" layer="51" font="vector" ratio="10" align="center"/>
 <attribute name="NAME" x="-30.75758125" y="12.00221875" size="1.27" layer="25" font="vector" ratio="10" align="center"/>
-<attribute name="NAME" x="-30.35758125" y="9.30221875" size="1.778" layer="51" font="vector" ratio="10" align="center"/>
 <attribute name="PIN1" value="" x="-33.39758125" y="16.24721875" size="1.778" layer="21" font="vector" rot="R90" align="center-left"/>
 <attribute name="PIN2" value="" x="-30.85758125" y="16.24721875" size="1.778" layer="21" font="vector" rot="R90" align="center-left"/>
@@
 <attribute name="VALUE" x="-59.370321875" y="30.318259375" size="1.2" layer="27" font="vector" ratio="10" rot="R90"/>
 </element>
-<element name="R10" library="quadparts_prebuilt" package="RESC2012X60_HS" value="2K" x="-56.324840625" y="35.10916875" smashed="yes" rot="R180">
-<attribute name="CREATOR" value="Swanson" x="-56.324840625" y="35.10916875" size="1.778" layer="27" rot="R180" display="off"/>
+<element name="R10" library="quadparts_prebuilt" package="RESC2012X60_HS" value="2.2K" x="-56.324840625" y="35.10916875" smashed="yes" rot="R180">
 <attribute name="DIST" value="DIGIKEY" x="-56.324840625" y="35.10916875" size="1.778" layer="27" rot="R180" display="off"/>
-<attribute name="DISTPN" value="311-2.0KARCT-ND" x="-56.324840625" y="35.10916875" size="1.778" layer="27" rot="R180" display="off"/>
+<attribute name="DISTPN" value="YAG3776CT-ND " x="-56.324840625" y="35.10916875" size="1.778" layer="27" rot="R180" display="off"/>
 <attribute name="NAME" x="-50.923571875" y="35.73648125" size="1.27" layer="25" font="vector" rot="R180"/>
-<attribute name="VALUE" x="-55.124840625" y="35.70916875" size="1.2" layer="27" font="vector" ratio="10" rot="R180"/>
+<attribute name="VALUE" value="2.2K" x="-55.124840625" y="35.70916875" size="1.2" layer="27" font="vector" ratio="10" rot="R180"/>
 </element>
 <element name="R11" library="quadparts_prebuilt" package="RESC2012X60_HS" value="270" x="-62.917478125" y="50.898940625" smashed="yes">
@@
 <attribute name="DIST" value="DIGIKEY" x="-49.4" y="4.9" size="1.778" layer="27" display="off"/>
 <attribute name="DISTPN" value="401-1999-1-ND" x="-49.4" y="4.9" size="1.778" layer="27" display="off"/>
-</element>
-<element name="R2" library="quadparts_prebuilt" package="RESC2012X60_HS" value="10K" x="-36.824640625" y="32.58041875" smashed="yes" rot="R180">
-<attribute name="CREATOR" value="Swanson" x="-36.824640625" y="32.58041875" size="1.778" layer="27" rot="R180" display="off"/>
-<attribute name="DIST" value="Digikey" x="-36.824640625" y="32.58041875" size="1.778" layer="27" rot="R180" display="off"/>
-<attribute name="DISTPN" value="311-10KARCT-ND" x="-36.824640625" y="32.58041875" size="1.778" layer="27" rot="R180" display="off"/>
-<attribute name="MFR" value="Yageo" x="-36.824640625" y="32.58041875" size="1.778" layer="27" rot="R180" display="off"/>
-<attribute name="MPN" value="RC0805JR-0710KL" x="-36.824640625" y="32.58041875" size="1.778" layer="27" rot="R180" display="off"/>
-<attribute name="NAME" x="-38.724640625" y="33.18041875" size="1.27" layer="25" font="vector" rot="R180"/>
-<attribute name="REVIEWER" value="Swanson" x="-36.824640625" y="32.58041875" size="1.778" layer="27" rot="R180" display="off"/>
-<attribute name="VALUE" x="-35.424640625" y="33.18041875" size="1.2" layer="27" font="vector" ratio="10" rot="R180"/>
 </element>
 <element name="D1" library="quadparts_prebuilt" package="SOD3716X135_HS" value="360mV" x="-63.821959375" y="31.252428125" smashed="yes" rot="R270">
@@
 <vertex x="-74.5" y="61.25"/>
 </polygon>
+<contactref element="R10" pad="2"/>
 <wire x1="-62.70458125" y1="11.1204625" x2="-70.25" y2="4.6" width="0" layer="19" extent="1-1"/>
 <wire x1="-51" y1="18.82" x2="-62.70458125" y2="11.1204625" width="0" layer="19" extent="1-1"/>
@@
 <wire x1="-50.720321875" y1="34.568259375" x2="-52.220321875" y2="33.213259375" width="0" layer="19" extent="1-1"/>
 <wire x1="-53.720321875" y1="36.568259375" x2="-50.720321875" y2="34.568259375" width="0" layer="19" extent="1-1"/>
-<wire x1="-58.970321875" y1="36.568259375" x2="-53.720321875" y2="36.568259375" width="0" layer="19" extent="1-1"/>
-<wire x1="-61.470321875" y1="34.818259375" x2="-58.970321875" y2="36.568259375" width="0" layer="19" extent="1-1"/>
-<wire x1="-59.970321875" y1="33.213259375" x2="-61.470321875" y2="34.818259375" width="0" layer="19" extent="1-1"/>
-<wire x1="-57.520421875" y1="32.318259375" x2="-59.970321875" y2="33.213259375" width="0" layer="19" extent="1-1"/>
+<wire x1="-57.279840625" y1="35.10916875" x2="-53.720321875" y2="36.568259375" width="0" layer="19" extent="1-1"/>
+<wire x1="-58.970321875" y1="36.568259375" x2="-57.279840625" y2="35.10916875" width="0" layer="19" extent="1-1"/>
+<wire x1="-57.520421875" y1="32.318259375" x2="-57.279840625" y2="35.10916875" width="0" layer="19" extent="1-1"/>
+<wire x1="-59.970321875" y1="33.213259375" x2="-57.520421875" y2="32.318259375" width="0" layer="19" extent="1-1"/>
+<wire x1="-61.470321875" y1="34.818259375" x2="-59.970321875" y2="33.213259375" width="0" layer="19" extent="1-1"/>
 <wire x1="-57.92384375" y1="43.5197" x2="-58.970321875" y2="36.568259375" width="0" layer="19" extent="1-1"/>
 <wire x1="-58.1962625" y1="46.76085625" x2="-57.92384375" y2="43.5197" width="0" layer="19" extent="1-1"/>
@@
 <contactref element="C13" pad="1"/>
 <contactref element="U3" pad="4"/>
-<contactref element="R2" pad="1"/>
 <contactref element="R11" pad="2"/>
 <contactref element="V11" pad="P1"/>
@@
 <wire x1="-30.85758125" y1="14.34221875" x2="-33.39758125" y2="14.34221875" width="0" layer="19" extent="1-1"/>
 <wire x1="-28.31758125" y1="14.34221875" x2="-30.85758125" y2="14.34221875" width="0" layer="19" extent="1-1"/>
-<wire x1="-35.869640625" y1="32.58041875" x2="-33.39758125" y2="14.34221875" width="0" layer="19" extent="1-1"/>
-<wire x1="-30.405428125" y1="36.591509375" x2="-35.869640625" y2="32.58041875" width="0" layer="19" extent="1-1"/>
+<wire x1="-70.2" y1="29.8" x2="-56.96118125" y2="15.6704625" width="0" layer="19" extent="1-1"/>
+<wire x1="-30.405428125" y1="36.591509375" x2="-30.85758125" y2="14.34221875" width="0" layer="19" extent="1-1"/>
 <wire x1="-37.717428125" y1="41.791509375" x2="-30.405428125" y2="36.591509375" width="0" layer="19" extent="1-1"/>
 <wire x1="-40.39708125" y1="40.96444375" x2="-37.717428125" y2="41.791509375" width="0" layer="19" extent="1-1"/>
-<wire x1="-70.2" y1="29.8" x2="-56.96118125" y2="15.6704625" width="0" layer="19" extent="1-1"/>
 <wire x1="-61.962478125" y1="50.898940625" x2="-70.2" y2="29.8" width="0" layer="19" extent="1-1"/>
 </signal>
@@
 <wire x1="-30.6" y1="48" x2="-45.4" y2="44.4" width="0" layer="19" extent="1-1"/>
 </signal>
-<signal name="CHR_ENABLE#">
-<contactref element="R10" pad="2"/>
-<contactref element="U3" pad="14"/>
-<contactref element="R2" pad="2"/>
-<wire x1="-37.779640625" y1="32.58041875" x2="-57.279840625" y2="35.10916875" width="0" layer="19" extent="1-1"/>
-<wire x1="-30.405428125" y1="43.091509375" x2="-37.779640625" y2="32.58041875" width="0" layer="19" extent="1-1"/>
-</signal>
 <signal name="N$15" class="1">

Commit message: verified 3.7V opertaion of ftdi regulator.  checked circuit on bread board
Parts:
- removed J4, J5: (no value), Components:HDRV3W63P254_3X1_762X254H838_HS
Connections:
- net BPOS: no longer J5.1
- net GND: no longer J5.3
- net N$11: no longer J4.1
- net N$12: no longer J5.2
- net VBUS: no longer J4.3
