File: hardware/controller_board_minimal.sch (EAGLE design)
At the start: 59 parts, among them J4 AVR_SPI_PRG_6NS, J8 FRSKY-GIMBAL-2X-SERVO, J9 FRSKY-GIMBAL-2X-SERVO, P1 TEST-POINT, P2 TEST-POINT, P3 TEST-POINT, P4 TEST-POINT, U1 ATMEGA128RFA1, U5 3.3V, Y1 CRYSTAL5X3

Commit message: notes from undergrads.  Tweak stencil fiducial. Some new parts
Parts:
- added E1: ROTARY-ENCODER-W/BUTTON-BOURNS-PEC12R-30MM, RemoteParts:ROTARY-ENCODER-W/BUTTON-BOURNS-PEC12R-30MM
- added U$4: NAV-SWITCH, RemoteParts:NAV-SWITCH
Changed lines of the file:
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@@
 <setting verticaltext="up"/>
 </settings>
-<grid distance="0.05" unitdist="inch" unit="inch" style="lines" multiple="1" display="no" altdistance="0.01" altunitdist="inch" altunit="inch"/>
+<grid distance="0.1" unitdist="inch" unit="inch" style="lines" multiple="1" display="no" altdistance="0.01" altunitdist="inch" altunit="inch"/>
 <layers>
 <layer number="99" name="SpiceOrder" color="7" fill="1" visible="no" active="no"/>
@@
 <part name="U$3" library="RemoteParts" deviceset="MOUNTING-HOLE" device="-M2.5-GROUNDED"/>
 <part name="U$6" library="RemoteParts" deviceset="MOUNTING-HOLE" device="-M2.5-GROUNDED"/>
+<part name="E1" library="RemoteParts" deviceset="ROTARY-ENCODER-W/BUTTON" device="-BOURNS-PEC12R-30MM"/>
+<part name="U$4" library="RemoteParts" deviceset="NAV-SWITCH" device=""/>
 </parts>
 <sheets>
@@
 <instance part="U$3" gate="G$1" x="302.26" y="267.97"/>
 <instance part="U$6" gate="G$1" x="312.42" y="267.97"/>
+<instance part="E1" gate="G$1" x="383.54" y="241.3"/>
+<instance part="U$4" gate="G$1" x="355.6" y="213.36"/>
 </instances>
 <busses>
