File: hardware/controller_board3.sch (EAGLE design)
At the start: 80 parts, among them J1 USB-MICROA-AMPHENOL-10118192-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, J2 2.4K, J3 2.4K, J4 AVR_SPI_PRG_6-SMD, J5 FTDI_BASIC-SMD, J6 FTDI-4PIN-RIGHT-ANGLE-SMD, J7 FRSKY-GIMBAL-2X-SERVO-SMD, J8 FRSKY-GIMBAL-2X-SERVO-SMD, P1 TEST-POINT, P2 TEST-POINT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

Commit message: passes eaglint
Parts:
- removed J5: FTDI_BASIC-SMD, quadparts_prebuilt:FTDI_BASIC-SMD
- removed J6: FTDI-4PIN-RIGHT-ANGLE-SMD, quadparts_prebuilt:FTDI-4PIN-RIGHT-ANGLE-SMD
- removed R1: 2.2K, quadparts_prebuilt:RESISTOR-PACK-4X-2.2K
- removed R3: 10K, quadparts_prebuilt:RESISTOR-PACK-4X-10K
- added JP1: FTDI_BASIC-SMD-REV, quadparts_prebuilt:FTDI_BASIC-SMD-REV
- added R2: 10K, quadparts_prebuilt:RESISTOR_SMD-2012-0805-10K
- added R7: 2.2K, quadparts_prebuilt:RESISTOR_SMD-2012-0805-2.2K
- added R8: 1.2K, quadparts_prebuilt:RESISTOR_SMD-2012-0805-1.2K
- added V9: LOCKED-VIA-0.2, quadparts_prebuilt:LOCKED-VIA-0.2
- A1: value ANTENNA-BOARD-REV -> ANTENNA-CHIP; device quadparts_prebuilt:ANTENNA-BOARD-REV -> quadparts_prebuilt:ANTENNA-CHIP
- B1, B10, B4, B5, B6, B7, B8, B9, C5, C6, C7, J7, J8: SUBSTITUTE_OK yes -> (none)
- B3: value BATTERY-SMD -> BATTERY; device quadparts_prebuilt:BATTERY-SMD -> quadparts_prebuilt:BATTERY
- C1, C8, C9: device quadparts_prebuilt:CAPACITOR-NP_SMD-0603_CERAMIC-0.1UF -> quadparts_prebuilt:CAPACITOR-NP_SMD-2012-0805_CERAMIC-0.1UF; SUBSTITUTE_OK yes -> (none)
- C11, C12, C13, C16, C4: device quadparts_prebuilt:CAPACITOR-NP_SMD-0603_CERAMIC-1UF -> quadparts_prebuilt:CAPACITOR-NP_SMD-2012-0805_CERAMIC-1UF; SUBSTITUTE_OK yes -> (none)
- C14, C15: device quadparts_prebuilt:CAPACITOR-NP_SMD-0603_CERAMIC-12PF -> quadparts_prebuilt:CAPACITOR-NP_SMD-2012-0805_CERAMIC-12PF
- C2: device quadparts_prebuilt:CAPACITOR-NP_SMD-0603_CERAMIC-0.75PF -> quadparts_prebuilt:CAPACITOR-NP_SMD-2012-0805_CERAMIC-0.75PF
- C3: device quadparts_prebuilt:CAPACITOR-NP_SMD-0603_CERAMIC-22PF -> quadparts_prebuilt:CAPACITOR-NP_SMD-2012-0805_CERAMIC-22PF
- D2, D3: device quadparts_prebuilt:DIODE-SCHOTTKY_-SMD-SOD123 -> quadparts_prebuilt:DIODE-SCHOTTKY_SMD-SOD123-360MV
- E1, J2, J3, P2, P3, P4: POPULATE NO -> (none)
- P1: POPULATE no -> (none)
- R4, R5: value 1.5K -> 750; device quadparts_prebuilt:RESISTOR-PACK-4X-1.5K -> quadparts_prebuilt:RESISTOR-PACK-4X-750; SUBSTITUTE_OK yes -> (none)
- S1, S2: value SWITCH-DPDT-300MA-6V-SMD -> POWER-SWITCH-MFS201N-9-Z-SMD-VERTICAL; device RemoteParts:SWITCH-DPDT-300MA-6V-SMD -> RemoteParts:POWER-SWITCH-MFS201N-9-Z-SMD-VERTICAL
- Y1: value CRYSTAL-SMD-3X2 -> CRYSTAL5X3; device quadparts_prebuilt:CRYSTAL-SMD-3X2 -> quadparts_prebuilt:CRYSTAL5X3
Connections:
- removed net BAT_SENSE: R1G$3.2, R3G$2.1, U4.PF7(ADC7/TDI)
- removed net N$14: D2.A, S1.ON1
- removed net VIN: C7.1, C8.1, D2.C, D3.C, J4.2, L1.VIN, P2.T, U3.VCC
- new net VREG_IN: C7.1, C8.1, L1.VIN, S1.ON, U3.VCC
- net 3V3: now also D4.A2, J4.2, JP1.4, R2.2, R8.2; no longer D4.A1, J5.4, R1G$1.2, R3G$4.2
- net BPOS: now also D3.A; no longer S1.C
- net CTS-1: now also JP1.5; no longer J5.5
- net DTR-1: now also JP1.1; no longer J5.1, J6.3
- net GND: now also JP1.6, R7.2, V9.N; no longer J5.6, J6.4, R1G$2.1, R1G$3.1, R3G$1.1
- net GREF: now also R8.1; no longer R1G$1.1
- net N$12: now also R7.1; no longer R1G$2.2
- net RESET: now also R2.1; no longer R3G$4.1
- net RF: now also D4.A1; no longer D4.A2
- net RXI-1: now also JP1.2; no longer J5.2, J6.1
- net TXO-1: now also JP1.3; no longer J5.3, J6.2
- net VBAT: now also D2.C, D3.C, P2.T, S1.C; no longer D3.A, R3G$2.2, S1.ON
- net VBUS: now also D2.A; no longer R3G$1.2, S1.C1
Other:
- note removed: "FTDI"
- note removed: "If the input to the charger floats, the battery leaks, so pull it down."
- note removed: "Use DPDT here so that 1) 'off' means off even when on USB and 2) there's no leakage through the voltage divider when when we are "off" Otherwise we'll deeply dischange the battery."
- moved on the sheet: B3, C12, C16, C5, D2, D3, P4
