File: hardware/releases/v4-rev6-rc1/controller_board.brd (EAGLE design)
At the start: 86 x 70 mm, 94 parts, among them J1 USB-MICROA-AMPHENOL-10118192-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, J2 2.4K, J3 2.4K, J4 AVR_SPI_PRG_6-SMD, J7 FRSKY-GIMBAL-2X-SERVO-SMD, J8 FRSKY-GIMBAL-2X-SERVO-SMD, P1 TEST-POINT, P2 TEST-POINT, P3 TEST-POINT, P4 TEST-POINT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

Commit message: update layout
Parts:
- moved U$5 108.6 mm to (40.0, -61.0)
- moved U$4 105.0 mm to (-46.1, -85.5)
- moved D2 0.71 mm to (-26.0, 12.0)
Connections:
- net BTN1/SCL renamed BTN1
- net BTN2/SDA renamed BTN2
- removed net BAT_SENSE: U4.3
- removed net CTS-0: U5.3
Routing:
- net VBUS: track 144.3 -> 0.00 mm
- net GREF: track 130.5 -> 0.00 mm, vias 1 -> 0
- net YAW: track 102.4 -> 0.00 mm, vias 3 -> 0
- net VBAT: track 104.0 -> 3.34 mm, vias 0 -> 3
- net BTN_LEFT: track 90.1 -> 0.00 mm, vias 2 -> 0
- net THROTTLE: track 88.9 -> 0.00 mm, vias 3 -> 0
- net ROLL: track 86.2 -> 0.00 mm
- net PROG_SEL: track 86.0 -> 0.00 mm, vias 2 -> 0
- net RESET: track 86.0 -> 0.00 mm, vias 3 -> 0
- net VREG_IN: track 84.1 -> 0.00 mm
- net E1-A: track 81.0 -> 0.00 mm, vias 1 -> 0
- net BTN_UP: track 79.7 -> 0.00 mm, vias 2 -> 0
- net E1-B: track 79.3 -> 0.00 mm, vias 1 -> 0
- net TXLED: track 72.8 -> 0.00 mm, vias 2 -> 0
- net BTN_RIGHT: track 67.2 -> 0.00 mm, vias 2 -> 0
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Other:
- board text added: "FTDI RX"
- board text added: "FTDI TX"
- board text added: "RF RX/TX"
- board text removed: "FTDI"
- board text removed: "RX/TX"
