File: hardware/releases/v4-rev6-rc1/controller_board.sch (EAGLE design)
At the start: 88 parts, among them J1 USB-MICROA-AMPHENOL-10118192-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, J2 2.4K, J3 2.4K, J4 AVR_SPI_PRG_6-SMD, J7 FRSKY-GIMBAL-2X-SERVO-SMD, J8 FRSKY-GIMBAL-2X-SERVO-SMD, P1 TEST-POINT, P2 TEST-POINT, P3 TEST-POINT, P4 TEST-POINT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

Commit message: update layout
Connections:
- net BTN1/SCL renamed BTN1
- net BTN2/SDA renamed BTN2
- removed net BAT_SENSE: U4.PF4(ADC4/TCK)
- removed net CTS-0: U5.1Y0
Other:
- moved on the sheet: JP1
Changed lines of the file:
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@@
 <setting verticaltext="up"/>
 </settings>
-<grid distance="0.05" unitdist="inch" unit="inch" style="lines" multiple="1" display="no" altdistance="0.01" altunitdist="inch" altunit="inch"/>
+<grid distance="0.1" unitdist="inch" unit="inch" style="lines" multiple="1" display="no" altdistance="0.01" altunitdist="inch" altunit="inch"/>
 <layers>
 <layer number="99" name="SpiceOrder" color="7" fill="1" visible="no" active="no"/>
@@
 <attribute name="VALUE" x="280.67" y="236.22" size="1.778" layer="96"/>
 </instance>
-<instance part="JP1" gate="G$1" x="422.91" y="64.77" smashed="yes" rot="R180">
-<attribute name="VALUE" x="427.99" y="74.93" size="1.778" layer="96" rot="R180"/>
-<attribute name="NAME" x="427.99" y="53.848" size="1.778" layer="95" rot="R180"/>
+<instance part="JP1" gate="G$1" x="384.81" y="62.23" smashed="yes" rot="R180">
+<attribute name="VALUE" x="389.89" y="72.39" size="1.778" layer="96" rot="R180"/>
+<attribute name="NAME" x="389.89" y="51.308" size="1.778" layer="95" rot="R180"/>
 </instance>
 <instance part="V9" gate="G$1" x="166.37" y="16.51" smashed="yes" rot="R90">
@@
 </segment>
 <segment>
-<label x="411.48" y="57.15" size="1.27" layer="95" rot="R180" xref="yes"/>
+<label x="373.38" y="54.61" size="1.27" layer="95" rot="R180" xref="yes"/>
 <pinref part="JP1" gate="G$1" pin="6"/>
-<wire x1="417.83" y1="57.15" x2="411.48" y2="57.15" width="0.1524" layer="91"/>
+<wire x1="379.73" y1="54.61" x2="373.38" y2="54.61" width="0.1524" layer="91"/>
 </segment>
 <segment>
@@
 </segment>
 <segment>
-<label x="411.48" y="62.23" size="1.27" layer="95" rot="R180" xref="yes"/>
+<label x="373.38" y="59.69" size="1.27" layer="95" rot="R180" xref="yes"/>
 <pinref part="JP1" gate="G$1" pin="4"/>
-<wire x1="417.83" y1="62.23" x2="411.48" y2="62.23" width="0.1524" layer="91"/>
+<wire x1="379.73" y1="59.69" x2="373.38" y2="59.69" width="0.1524" layer="91"/>
 </segment>
 <segment>
@@
 <net name="DTR-1" class="0">
 <segment>
-<label x="411.48" y="69.85" size="1.27" layer="95" rot="R180" xref="yes"/>
+<label x="373.38" y="67.31" size="1.27" layer="95" rot="R180" xref="yes"/>
 <pinref part="JP1" gate="G$1" pin="1"/>
-<wire x1="417.83" y1="69.85" x2="411.48" y2="69.85" width="0.1524" layer="91"/>
+<wire x1="379.73" y1="67.31" x2="373.38" y2="67.31" width="0.1524" layer="91"/>
 </segment>
 <segment>
@@
 <net name="RXI-1" class="0">
 <segment>
-<label x="411.48" y="67.31" size="1.27" layer="95" rot="R180" xref="yes"/>
+<label x="373.38" y="64.77" size="1.27" layer="95" rot="R180" xref="yes"/>
 <pinref part="JP1" gate="G$1" pin="2"/>
-<wire x1="417.83" y1="67.31" x2="411.48" y2="67.31" width="0.1524" layer="91"/>
+<wire x1="379.73" y1="64.77" x2="373.38" y2="64.77" width="0.1524" layer="91"/>
 </segment>
 <segment>
@@
 <net name="TXO-1" class="0">
 <segment>
-<label x="411.48" y="64.77" size="1.27" layer="95" rot="R180" xref="yes"/>
+<label x="373.38" y="62.23" size="1.27" layer="95" rot="R180" xref="yes"/>
 <pinref part="JP1" gate="G$1" pin="3"/>
-<wire x1="417.83" y1="64.77" x2="411.48" y2="64.77" width="0.1524" layer="91"/>
+<wire x1="379.73" y1="62.23" x2="373.38" y2="62.23" width="0.1524" layer="91"/>
 </segment>
 <segment>
@@
 <net name="CTS-1" class="0">
 <segment>
-<label x="411.48" y="59.69" size="1.27" layer="95" rot="R180" xref="yes"/>
+<label x="373.38" y="57.15" size="1.27" layer="95" rot="R180" xref="yes"/>
 <pinref part="JP1" gate="G$1" pin="5"/>
-<wire x1="417.83" y1="59.69" x2="411.48" y2="59.69" width="0.1524" layer="91"/>
+<wire x1="379.73" y1="57.15" x2="373.38" y2="57.15" width="0.1524" layer="91"/>
 </segment>
 <segment>
@@
 <wire x1="309.88" y1="111.76" x2="312.42" y2="111.76" width="0.1524" layer="91"/>
 <label x="312.42" y="111.76" size="1.27" layer="95" xref="yes"/>
-</segment>
-</net>
-<net name="CTS-0" class="0">
-<segment>
-<pinref part="U5" gate="G$1" pin="1Y0"/>
-<wire x1="309.88" y1="114.3" x2="312.42" y2="114.3" width="0.1524" layer="91"/>
-<label x="312.42" y="114.3" size="1.27" layer="95" xref="yes"/>
 </segment>
 </net>
@@
 </segment>
 </net>
-<net name="BAT_SENSE" class="0">
-<segment>
-<pinref part="U4" gate="G$1" pin="PF4(ADC4/TCK)"/>
-<wire x1="220.98" y1="184.15" x2="223.52" y2="184.15" width="0.1524" layer="91"/>
-<label x="223.52" y="184.15" size="1.27" layer="95" xref="yes"/>
-</segment>
-</net>
-<net name="BTN1/SCL" class="0">
+<net name="BTN1" class="0">
 <segment>
 <pinref part="U4" gate="G$1" pin="PD0(SCL/INT0)"/>
@@
 </segment>
 </net>
-<net name="BTN2/SDA" class="0">
+<net name="BTN2" class="0">
 <segment>
 <pinref part="U4" gate="G$1" pin="PD1(SDA/INT1)"/>
