File: LTC4063-test/ltc4063-test.brd (EAGLE design)
At the start: 38 x 34.5 mm, 18 parts, among them J1 USB-MICROA-AMPHENOL-10118192-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, P1 TEST-POINT, P2 TEST-POINT, P3 TEST-POINT, P4 TEST-POINT, P5 TEST-POINT, P6 TEST-POINT, U1 LIPO-VREG-LTC4063

Commit message: tweak board shape
Other:
- board size 38 x 34.5 mm -> 38 x 38 mm
Changed lines of the file:
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@@
 <board>
 <plain>
-<wire x1="0" y1="98" x2="0" y2="67.5" width="0.01" layer="20"/>
-<wire x1="0" y1="67.5" x2="2" y2="65.5" width="0.01" layer="20" curve="90"/>
-<wire x1="2" y1="65.5" x2="36" y2="65.5" width="0.01" layer="20"/>
-<wire x1="36" y1="65.5" x2="38" y2="67.5" width="0.01" layer="20" curve="90"/>
-<wire x1="38" y1="67.5" x2="38" y2="98" width="0.01" layer="20"/>
+<wire x1="0" y1="98" x2="0" y2="64" width="0.01" layer="20"/>
+<wire x1="0" y1="64" x2="2" y2="62" width="0.01" layer="20" curve="90"/>
+<wire x1="2" y1="62" x2="36" y2="62" width="0.01" layer="20"/>
+<wire x1="36" y1="62" x2="38" y2="64" width="0.01" layer="20" curve="90"/>
+<wire x1="38" y1="64" x2="38" y2="98" width="0.01" layer="20"/>
 <wire x1="38" y1="98" x2="36" y2="100" width="0.01" layer="20" curve="90"/>
 <wire x1="36" y1="100" x2="2" y2="100" width="0.01" layer="20"/>
@@
 <text x="25" y="72" size="1.778" layer="21" font="vector" rot="R90" align="center-right">VBUS</text>
 <text x="36" y="80" size="1.3" layer="21" font="vector" align="center-right">Steven Swanson</text>
-<text x="30" y="69" size="1.3" layer="21" font="vector" align="center-left">LTC4063
+<text x="30" y="65.5" size="1.3" layer="21" font="vector" align="center-left">LTC4063
 breakout
 rev0</text>
 <hole x="5" y="90" drill="3.2"/>
 <hole x="5" y="97" drill="3.2"/>
+<dimension x1="2" y1="100" x2="2" y2="62" x3="-3" y3="81" textsize="0.9" layer="47"/>
+<dimension x1="0" y1="64" x2="38" y2="64" x3="19" y3="60.5" textsize="0.9" layer="47"/>
 </plain>
 <attributes>
@@
 <polygon width="0.1524" layer="1">
 <vertex x="-1" y="101"/>
-<vertex x="-1" y="64"/>
-<vertex x="39" y="64"/>
+<vertex x="-1" y="60.5"/>
+<vertex x="39" y="60.5"/>
 <vertex x="39" y="101"/>
 </polygon>
@@
 <polygon width="0.1524" layer="16">
 <vertex x="-2" y="102"/>
-<vertex x="-2" y="63"/>
-<vertex x="40" y="63"/>
+<vertex x="-2" y="59.5"/>
+<vertex x="40" y="59.5"/>
 <vertex x="40" y="102"/>
 </polygon>

Commit message: small tweaks
Parts:
- R1: value 33K -> 30K
Routing:
- net N$1: track 43.3 -> 54.1 mm
- net VBUS: track 41.0 -> 38.4 mm
- net FB\: track 18.1 -> 20.5 mm
- net N$5: track 7.69 -> 9.92 mm
- net PROG: track 21.8 -> 23.4 mm
- net VBAT: track 42.1 -> 43.3 mm
- net 3V3: track 19.2 -> 18.5 mm
Other:
- board text added: "3V3"
- board text added: "LTC4063 test board rev0"
- board text removed: "3v3"
- board text removed: "LTC4063 breakout rev0"
