File: LTC4063-test/ltc4063-test.sch (EAGLE design)
At the start: 17 parts, among them J1 USB-MICROA-AMPHENOL-10118192-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, P1 TEST-POINT, P2 TEST-POINT, P3 TEST-POINT, P4 TEST-POINT, P5 TEST-POINT, P6 TEST-POINT, U1 LIPO-VREG-LTC4063

Commit message: small tweaks
Parts:
- R1: value 33K -> 30K; device quadparts_prebuilt:RESISTOR_SMD-2012-0805-33K -> quadparts_prebuilt:RESISTOR_SMD-2012-0805-30K
Other:
- moved on the sheet: J1, P1
Changed lines of the file:
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@@
 <setting verticaltext="up"/>
 </settings>
-<grid distance="0.1" unitdist="inch" unit="inch" style="lines" multiple="1" display="no" altdistance="0.01" altunitdist="inch" altunit="inch"/>
+<grid distance="0.05" unitdist="inch" unit="inch" style="lines" multiple="1" display="no" altdistance="0.01" altunitdist="inch" altunit="inch"/>
 <layers>
 <layer number="1" name="Top" color="4" fill="1" visible="no" active="no"/>
@@
 <layer number="91" name="Nets" color="2" fill="1" visible="yes" active="yes"/>
 <layer number="92" name="Busses" color="1" fill="1" visible="yes" active="yes"/>
-<layer number="93" name="Pins" color="2" fill="1" visible="yes" active="yes"/>
+<layer number="93" name="Pins" color="2" fill="1" visible="no" active="yes"/>
 <layer number="94" name="Symbols" color="4" fill="1" visible="yes" active="yes"/>
 <layer number="95" name="Names" color="7" fill="1" visible="yes" active="yes"/>
@@
 <part name="J1" library="RemoteParts" deviceset="USB" device="-MICROA-AMPHENOL-10118192-0001LF"/>
 <part name="B1" library="quadparts_prebuilt" deviceset="BATTERY" device="-SPRING-SMD"/>
-<part name="GND1" library="quadparts_prebuilt" deviceset="GND" device=""/>
-<part name="GND2" library="quadparts_prebuilt" deviceset="GND" device=""/>
 <part name="P1" library="RemoteParts" deviceset="TEST-POINT" device=""/>
 <part name="P2" library="RemoteParts" deviceset="TEST-POINT" device=""/>
@@
 <part name="C1" library="quadparts_prebuilt" deviceset="CAPACITOR-NP_" device="SMD-2012-0805_CERAMIC-1UF" value="1uF"/>
 <part name="C2" library="quadparts_prebuilt" deviceset="CAPACITOR-NP_" device="SMD-2012-0805_CERAMIC-10UF" value="10uF"/>
-<part name="GND4" library="quadparts_prebuilt" deviceset="GND" device=""/>
-<part name="GND5" library="quadparts_prebuilt" deviceset="GND" device=""/>
-<part name="R1" library="quadparts_prebuilt" deviceset="RESISTOR_" device="SMD-2012-0805-33K" value="33K"/>
+<part name="R1" library="quadparts_prebuilt" deviceset="RESISTOR_" device="SMD-2012-0805-30K" value="30K"/>
 <part name="R2" library="quadparts_prebuilt" deviceset="RESISTOR_" device="SMD-2012-0805-10K" value="10K"/>
-<part name="GND6" library="quadparts_prebuilt" deviceset="GND" device=""/>
 <part name="D1" library="quadparts_prebuilt" deviceset="DIODE-LED_" device="SMD-2012-0805-GREEN" value="green"/>
 <part name="R3" library="quadparts_prebuilt" deviceset="RESISTOR_" device="SMD-2012-0805-270" value="270"/>
@@
 </instance>
 <instance part="U1" gate="G$1" x="179.07" y="182.88" smashed="yes"/>
-<instance part="J1" gate="A" x="101.6" y="207.01" smashed="yes" rot="R180">
-<attribute name="NAME" x="96.52" y="214.63" size="1.27" layer="95" font="vector" rot="R180" align="top-center"/>
-</instance>
-<instance part="B1" gate="G$1" x="215.9" y="193.04" smashed="yes">
-<attribute name="NAME" x="208.28" y="198.12" size="1.778" layer="95" font="vector"/>
-</instance>
-<instance part="GND1" gate="1" x="123.19" y="209.55" smashed="yes">
-<attribute name="VALUE" x="123.19" y="207.01" size="1.778" layer="96" align="center"/>
-</instance>
-<instance part="GND2" gate="1" x="229.87" y="190.5" smashed="yes">
-<attribute name="VALUE" x="229.87" y="187.96" size="1.778" layer="96" align="center"/>
-</instance>
-<instance part="P1" gate="G$1" x="227.33" y="193.04" smashed="yes">
-<attribute name="NAME" x="227.33" y="200.66" size="1.27" layer="95" align="center"/>
+<instance part="J1" gate="A" x="119.38" y="187.96" smashed="yes" rot="MR0">
+<attribute name="NAME" x="114.3" y="180.34" size="1.27" layer="95" font="vector" rot="MR0" align="top-center"/>
+</instance>
+<instance part="B1" gate="G$1" x="218.44" y="176.53" smashed="yes" rot="R270">
+<attribute name="NAME" x="220.98" y="180.34" size="1.778" layer="95" font="vector"/>
+</instance>
+<instance part="P1" gate="G$1" x="218.44" y="162.56" smashed="yes" rot="R180">
+<attribute name="NAME" x="218.44" y="154.94" size="1.27" layer="95" rot="R180" align="center"/>
 </instance>
 <instance part="P2" gate="G$1" x="204.47" y="190.5" smashed="yes">
@@
 <attribute name="NAME" x="201.422" y="185.039" size="1.778" layer="95" rot="R180"/>
 </instance>
-<instance part="GND4" gate="1" x="201.93" y="180.34" smashed="yes">
-<attribute name="VALUE" x="201.93" y="177.8" size="1.778" layer="96" align="center"/>
-</instance>
-<instance part="GND5" gate="1" x="134.62" y="182.88" smashed="yes">
-<attribute name="VALUE" x="134.62" y="180.34" size="1.778" layer="96" align="center"/>
-</instance>
 <instance part="R1" gate="G$1" x="194.31" y="185.42" smashed="yes" rot="R90">
 <attribute name="VALUE" x="197.612" y="181.61" size="1.778" layer="96" rot="R90"/>
@@
 <attribute name="VALUE" x="197.612" y="166.37" size="1.778" layer="96" rot="R90"/>
 <attribute name="NAME" x="192.8114" y="166.37" size="1.778" layer="95" rot="R90"/>
-</instance>
-<instance part="GND6" gate="1" x="194.31" y="162.56" smashed="yes">
-<attribute name="VALUE" x="194.31" y="160.02" size="1.778" layer="96" align="center"/>
 </instance>
 <instance part="D1" gate="G$1" x="158.75" y="190.5" smashed="yes">
@@
 <segment>
 <pinref part="J1" gate="A" pin="1-VCC"/>
-<wire x1="106.68" y1="201.93" x2="134.62" y2="201.93" width="0.1524" layer="91"/>
-<wire x1="134.62" y1="201.93" x2="134.62" y2="193.04" width="0.1524" layer="91"/>
 <pinref part="U1" gate="G$1" pin="VCC"/>
 <wire x1="134.62" y1="193.04" x2="143.51" y2="193.04" width="0.1524" layer="91"/>
@@
 <wire x1="143.51" y1="190.5" x2="143.51" y2="193.04" width="0.1524" layer="91"/>
 <junction x="143.51" y="193.04"/>
-<label x="134.62" y="201.93" size="1.27" layer="95" xref="yes"/>
+<label x="134.62" y="193.04" size="1.27" layer="95" xref="yes"/>
 <pinref part="P3" gate="G$1" pin="T"/>
 <junction x="146.05" y="193.04"/>
+<wire x1="124.46" y1="193.04" x2="134.62" y2="193.04" width="0.1524" layer="91"/>
 </segment>
 </net>
 <net name="GND" class="0">
 <segment>
-<pinref part="J1" gate="A" pin="5-GND"/>
-<pinref part="GND1" gate="1" pin="GND"/>
-<wire x1="106.68" y1="212.09" x2="123.19" y2="212.09" width="0.1524" layer="91"/>
-</segment>
-<segment>
 <pinref part="B1" gate="G$1" pin="N"/>
-<pinref part="GND2" gate="1" pin="GND"/>
-<wire x1="220.98" y1="193.04" x2="227.33" y2="193.04" width="0.1524" layer="91"/>
+<wire x1="218.44" y1="171.45" x2="218.44" y2="162.56" width="0.1524" layer="91"/>
 <pinref part="P1" gate="G$1" pin="T"/>
-<wire x1="227.33" y1="193.04" x2="229.87" y2="193.04" width="0.1524" layer="91"/>
-<junction x="227.33" y="193.04"/>
-</segment>
-<segment>
+<wire x1="218.44" y1="162.56" x2="201.93" y2="162.56" width="0.1524" layer="91"/>
 <pinref part="U1" gate="G$1" pin="GND"/>
 <pinref part="GND3" gate="1" pin="GND"/>
@@
 <wire x1="163.83" y1="177.8" x2="143.51" y2="177.8" width="0.1524" layer="91"/>
 <wire x1="143.51" y1="177.8" x2="143.51" y2="162.56" width="0.1524" layer="91"/>
-</segment>
-<segment>
+<pinref part="C1" gate="G$1" pin="1"/>
+<wire x1="134.62" y1="162.56" x2="134.62" y2="185.42" width="0.1524" layer="91"/>
+<wire x1="143.51" y1="162.56" x2="134.62" y2="162.56" width="0.1524" layer="91"/>
+<pinref part="R2" gate="G$1" pin="1"/>
+<wire x1="194.31" y1="162.56" x2="194.31" y2="165.1" width="0.1524" layer="91"/>
+<wire x1="163.83" y1="162.56" x2="194.31" y2="162.56" width="0.1524" layer="91"/>
+<junction x="194.31" y="162.56"/>
 <pinref part="C2" gate="G$1" pin="1"/>
-<pinref part="GND4" gate="1" pin="GND"/>
-</segment>
-<segment>
-<pinref part="C1" gate="G$1" pin="1"/>
-<pinref part="GND5" gate="1" pin="GND"/>
-</segment>
-<segment>
-<pinref part="R2" gate="G$1" pin="1"/>
-<pinref part="GND6" gate="1" pin="GND"/>
+<wire x1="201.93" y1="162.56" x2="201.93" y2="182.88" width="0.1524" layer="91"/>
+<wire x1="194.31" y1="162.56" x2="201.93" y2="162.56" width="0.1524" layer="91"/>
+<pinref part="J1" gate="A" pin="5-GND"/>
+<wire x1="124.46" y1="182.88" x2="124.46" y2="162.56" width="0.1524" layer="91"/>
+<wire x1="134.62" y1="162.56" x2="124.46" y2="162.56" width="0.1524" layer="91"/>
 </segment>
 </net>
@@
 <label x="196.85" y="193.04" size="1.27" layer="95" rot="R90" xref="yes"/>
 <pinref part="P5" gate="G$1" pin="T"/>
-<wire x1="199.39" y1="193.04" x2="208.28" y2="193.04" width="0.1524" layer="91"/>
+<wire x1="199.39" y1="193.04" x2="218.44" y2="193.04" width="0.1524" layer="91"/>
+<wire x1="218.44" y1="193.04" x2="218.44" y2="181.61" width="0.1524" layer="91"/>
 <junction x="199.39" y="193.04"/>
 </segment>

Commit message: support for new remote firmware features
Other:
- note added: "This design works fine."
Changed lines of the file:
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@@
 <setting verticaltext="up"/>
 </settings>
-<grid distance="0.05" unitdist="inch" unit="inch" style="lines" multiple="1" display="no" altdistance="0.01" altunitdist="inch" altunit="inch"/>
+<grid distance="0.1" unitdist="inch" unit="inch" style="lines" multiple="1" display="no" altdistance="0.01" altunitdist="inch" altunit="inch"/>
 <layers>
 <layer number="1" name="Top" color="4" fill="1" visible="no" active="no"/>
@@
 <sheet>
 <plain>
+<text x="160.02" y="200.66" size="1.778" layer="91">This design works fine.</text>
 </plain>
 <instances>
