File: multicharger/multicharger.sch (EAGLE design)
At the start: 28 parts, among them J2 USB-A-SMD-KEYSTONE-931, J3 HEADER-8POS-, P1 TEST-POINT-1MM, P2 TEST-POINT-1MM, P3 TEST-POINT-1MM, P4 TEST-POINT-1MM, P5 TEST-POINT-1MM, P6 TEST-POINT-1MM, P7 1K, P8 TEST-POINT-1MM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

Commit message: More compact design
Parts:
- added B1, B2, B3, B4: BATTERY-SMD, quadparts_prebuilt:BATTERY-SMD
Changed lines of the file:
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@@
 <part name="P8" library="RemoteParts" deviceset="TEST-POINT" device="-1MM" value="TEST-POINT-1MM"/>
 <part name="P9" library="RemoteParts" deviceset="TEST-POINT" device="-1MM" value="TEST-POINT-1MM"/>
+<part name="B1" library="quadparts_prebuilt" deviceset="BATTERY" device="-SMD"/>
+<part name="B2" library="quadparts_prebuilt" deviceset="BATTERY" device="-SMD"/>
+<part name="B3" library="quadparts_prebuilt" deviceset="BATTERY" device="-SMD"/>
+<part name="B4" library="quadparts_prebuilt" deviceset="BATTERY" device="-SMD"/>
 </parts>
 <sheets>
@@
 <attribute name="NAME" x="109.22" y="147.32" size="1.27" layer="95" align="center"/>
 </instance>
+<instance part="B1" gate="G$1" x="246.38" y="248.92" smashed="yes">
+<attribute name="NAME" x="245.11" y="254" size="1.778" layer="95" font="vector" align="center"/>
+</instance>
+<instance part="B2" gate="G$1" x="246.38" y="241.3" smashed="yes">
+<attribute name="NAME" x="245.11" y="246.38" size="1.778" layer="95" font="vector" align="center"/>
+</instance>
+<instance part="B3" gate="G$1" x="246.38" y="233.68" smashed="yes">
+<attribute name="NAME" x="245.11" y="238.76" size="1.778" layer="95" font="vector" align="center"/>
+</instance>
+<instance part="B4" gate="G$1" x="246.38" y="226.06" smashed="yes">
+<attribute name="NAME" x="245.11" y="231.14" size="1.778" layer="95" font="vector" align="center"/>
+</instance>
 </instances>
